File: e202var-receiver-v1.brd (EAGLE design)
At the start: 56.4 x 80.7 mm, 50 parts, among them J1 9V, J2 ON/OFF, J3 HEADPHONES, P10 10k, Q1 BC547, Q2 BC547, U1 MC7809, U2 TLE2426, U3 LM386, U4 TL081C

Commit message: Finished layout.
Parts:
- moved C6 2.30 mm to (41.7, 45.7), turned to 90 degrees
- moved C13 1.05 mm to (5.08, 40.1), turned to 90 degrees
Routing:
- net Q1OUT: track 0.00 -> 81.8 mm
- net 9V: track 0.00 -> 72.0 mm
- net 2V: track 0.00 -> 54.7 mm
- net N$21: track 0.00 -> 48.9 mm
- net N$6: track 0.00 -> 39.8 mm
- net N$8: track 0.00 -> 33.4 mm
- net N$17: track 0.00 -> 30.6 mm
- net N$23: track 0.00 -> 26.7 mm
- net N$7: track 0.00 -> 26.7 mm
- net N$14: track 0.00 -> 23.8 mm
- net N$13: track 0.00 -> 22.9 mm
- net N$19: track 0.00 -> 20.6 mm
- net VIN2: track 0.00 -> 19.8 mm
- net 9V1: track 0.00 -> 18.3 mm
- net VIN: track 0.00 -> 17.8 mm
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- added copper zone on layer 16, net 2V
Other:
- board text removed: "ROUTE 2V on BOTTOM"

Commit message: Added CAM, DRU, clean BOM, library, and final of everything. Now we wait for Oct 30th.
Parts:
- added H4: MOUNT-PAD-ROUND3.2, holes:3,2-PAD
- moved LAMP 0.51 mm to (36.6, 66.3)
Connections:
- net GND: now also H4.B3,2
Other:
- board text added: "E202VAR Receiver v1 Wickerbox Electronics"
- board text added: "jeh.wicker@gmail.com"
