File: e202var-receiver-v1.sch (EAGLE design)
At the start: 48 parts, among them J1 9V, J1ALT 9V, J2 ON/OFF, J3 HEADPHONES, P10 10k, Q1 BC547, Q2 BC547, U1 MC7809, U2 TLE2426, U3 LM386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

Commit message: Placed components. Board size probably 2.22x3.18 inches. 5.25 for three at OSH Park.
Parts:
- removed J1ALT: 9V, e202var-receiver:CONN-2PIN
- added H1, H2, H3: MOUNT-PAD-ROUND3.2, holes:MOUNT-PAD-ROUND3.2
Connections:
- net N$2 renamed 9V2
- net N$3 renamed VIN
- net N$4 renamed Q1OUT
- net N$5 renamed VIN2
- removed net N$1: J1.PWR, J1ALT.1, J2.2
- new net 9V1: J1.PWR, J2.2
- net GND: now also H1.MOUNT, H2.MOUNT, H3.MOUNT; no longer J1ALT.2
Other:
- note added: "9V Power Options ----------------- 1. Place a barrel jack in J1 2. Solder wires to J1 holes"
- note added: "AMPLIFIER"
- note removed: "9V Power Options ----------------- 1. Place a barrel jack in J1 2. Solder wires or a header to J1ALT holes"
Changed lines of the file:
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@@
 <layer number="95" name="Names" color="15" fill="1" visible="yes" active="yes"/>
 <layer number="96" name="Values" color="15" fill="1" visible="yes" active="yes"/>
-<layer number="97" name="Info" color="7" fill="1" visible="yes" active="yes"/>
+<layer number="97" name="Info" color="15" fill="1" visible="yes" active="yes"/>
 <layer number="98" name="Guide" color="6" fill="1" visible="yes" active="yes"/>
 <layer number="99" name="Invisibles" color="7" fill="1" visible="no" active="no"/>
@@
 <part name="J1" library="e202var-receiver" deviceset="JACK-POWER-BARREL" device="" value="9V"/>
 <part name="J2" library="e202var-receiver" deviceset="CONN-2PIN" device="" value="ON/OFF"/>
-<part name="J1ALT" library="e202var-receiver" deviceset="CONN-2PIN" device="" value="9V"/>
 <part name="R6" library="e202var-receiver" deviceset="RESISTOR" device="" value="100k"/>
 <part name="U$1" library="e202var-receiver" deviceset="SYM-GND" device=""/>
+<part name="H1" library="holes" deviceset="MOUNT-PAD-ROUND" device="3.2"/>
+<part name="H2" library="holes" deviceset="MOUNT-PAD-ROUND" device="3.2"/>
+<part name="H3" library="holes" deviceset="MOUNT-PAD-ROUND" device="3.2"/>
+<part name="U$2" library="e202var-receiver" deviceset="SYM-GND" device=""/>
 </parts>
 <sheets>
@@
    jack in J1
 2. Solder wires
-   or a header
-   to J1ALT holes</text>
+   to J1 holes</text>
 <text x="-2.54" y="152.4" size="1.778" layer="97">J2 holes for
 24AWG wires
@@
 Sometimes called Natural Radio</text>
 <frame x1="-12.7" y1="2.54" x2="335.28" y2="180.34" columns="8" rows="5" layer="94"/>
+<text x="266.7" y="104.14" size="1.778" layer="97">AMPLIFIER</text>
 </plain>
 <instances>
@@
 <instance part="J1" gate="G$1" x="5.08" y="121.92" rot="MR0"/>
 <instance part="J2" gate="G$1" x="0" y="142.24"/>
-<instance part="J1ALT" gate="G$1" x="38.1" y="121.92" rot="MR0"/>
 <instance part="R6" gate="G$1" x="48.26" y="81.28" rot="R270"/>
 <instance part="U$1" gate="G$1" x="297.18" y="66.04"/>
+<instance part="H1" gate="G$1" x="7.62" y="40.64"/>
+<instance part="H2" gate="G$1" x="7.62" y="33.02"/>
+<instance part="H3" gate="G$1" x="7.62" y="25.4"/>
+<instance part="U$2" gate="G$1" x="2.54" y="15.24"/>
 </instances>
 <busses>
 </busses>
 <nets>
-<net name="N$1" class="0">
+<net name="9V1" class="0">
 <segment>
 <wire x1="12.7" y1="124.46" x2="25.4" y2="124.46" width="0.1524" layer="91"/>
@@
 <pinref part="J1" gate="G$1" pin="PWR"/>
 <pinref part="J2" gate="G$1" pin="2"/>
-<pinref part="J1ALT" gate="G$1" pin="1"/>
-<wire x1="30.48" y1="124.46" x2="25.4" y2="124.46" width="0.1524" layer="91"/>
-<junction x="25.4" y="124.46"/>
-</segment>
-</net>
-<net name="N$2" class="0">
+</segment>
+</net>
+<net name="9V2" class="0">
 <segment>
 <wire x1="7.62" y1="144.78" x2="25.4" y2="144.78" width="0.1524" layer="91"/>
@@
 </segment>
 </net>
-<net name="N$5" class="0">
+<net name="VIN2" class="0">
 <segment>
 <pinref part="U1" gate="G$1" pin="IN"/>
@@
 </segment>
 </net>
-<net name="N$3" class="0">
+<net name="VIN" class="0">
 <segment>
 <pinref part="D2" gate="G$1" pin="ANODE"/>
@@
 <wire x1="12.7" y1="119.38" x2="25.4" y2="119.38" width="0.1524" layer="91"/>
 <junction x="25.4" y="119.38"/>
-<pinref part="J1ALT" gate="G$1" pin="2"/>
-<wire x1="30.48" y1="121.92" x2="25.4" y2="121.92" width="0.1524" layer="91"/>
-<junction x="25.4" y="121.92"/>
 <pinref part="R6" gate="G$1" pin="2"/>
 <wire x1="48.26" y1="76.2" x2="48.26" y2="71.12" width="0.1524" layer="91"/>
@@
 <wire x1="246.38" y1="121.92" x2="246.38" y2="119.38" width="0.1524" layer="91"/>
 </segment>
-</net>
-<net name="N$4" class="0">
+<segment>
+<pinref part="H1" gate="G$1" pin="MOUNT"/>
+<wire x1="5.08" y1="40.64" x2="2.54" y2="40.64" width="0.1524" layer="91"/>
+<wire x1="2.54" y1="40.64" x2="2.54" y2="33.02" width="0.1524" layer="91"/>
+<pinref part="H2" gate="G$1" pin="MOUNT"/>
+<wire x1="2.54" y1="33.02" x2="5.08" y2="33.02" width="0.1524" layer="91"/>
+<junction x="2.54" y="33.02"/>
+<wire x1="2.54" y1="33.02" x2="2.54" y2="25.4" width="0.1524" layer="91"/>
+<wire x1="2.54" y1="25.4" x2="2.54" y2="15.24" width="0.1524" layer="91"/>
+<pinref part="H3" gate="G$1" pin="MOUNT"/>
+<wire x1="5.08" y1="25.4" x2="2.54" y2="25.4" width="0.1524" layer="91"/>
+<junction x="2.54" y="25.4"/>
+<pinref part="U$2" gate="G$1" pin="GND"/>
+</segment>
+</net>
+<net name="Q1OUT" class="0">
 <segment>
 <pinref part="Q1" gate="G$1" pin="B"/>

Commit message: Added CAM, DRU, clean BOM, library, and final of everything. Now we wait for Oct 30th.
Parts:
- added H4: MOUNT-PAD-ROUND3.2, holes:MOUNT-PAD-ROUND3.2
Connections:
- net GND: now also H4.MOUNT
Changed lines of the file:
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@@
 <part name="H3" library="holes" deviceset="MOUNT-PAD-ROUND" device="3.2"/>
 <part name="U$2" library="e202var-receiver" deviceset="SYM-GND" device=""/>
+<part name="H4" library="holes" deviceset="MOUNT-PAD-ROUND" device="3.2"/>
 </parts>
 <sheets>
@@
 <instance part="H3" gate="G$1" x="7.62" y="25.4"/>
 <instance part="U$2" gate="G$1" x="2.54" y="15.24"/>
+<instance part="H4" gate="G$1" x="7.62" y="17.78"/>
 </instances>
 <busses>
@@
 <junction x="2.54" y="33.02"/>
 <wire x1="2.54" y1="33.02" x2="2.54" y2="25.4" width="0.1524" layer="91"/>
-<wire x1="2.54" y1="25.4" x2="2.54" y2="15.24" width="0.1524" layer="91"/>
+<wire x1="2.54" y1="25.4" x2="2.54" y2="17.78" width="0.1524" layer="91"/>
 <pinref part="H3" gate="G$1" pin="MOUNT"/>
+<wire x1="2.54" y1="17.78" x2="2.54" y2="15.24" width="0.1524" layer="91"/>
 <wire x1="5.08" y1="25.4" x2="2.54" y2="25.4" width="0.1524" layer="91"/>
 <junction x="2.54" y="25.4"/>
 <pinref part="U$2" gate="G$1" pin="GND"/>
-</segment>
-</net>
+<wire x1="5.08" y1="17.78" x2="2.54" y2="17.78" width="0.1524" layer="91"/>
+<junction x="2.54" y="17.78"/>
+<pinref part="H4" gate="G$1" pin="MOUNT"/>
+</segment>
+</net>
