File: e202var-vlf-radio-receiver.kicad_pcb (KiCad board)
At the start: 2 copper layers, 55.9 x 81.3 mm, 52 parts, among them J1 9V, J2 ON/OFF, J3 HEADPHONES, J4 12V/18V, J5 FILTER, Q1 BC547, Q2 BC547, U1 MC7809, U2 TLE2426, U3 NJM386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

Commit message: v1.3 fixes in place. Saving before running script.
Parts:
- added C13 (x20): 100uF, Wickerlib:CAP-DISC-D7.5MM-P5MM, F.Cu at (62.7, 69.1)
- added R14: 2.2K, Wickerlib:RES-CARBONFILM-7MM, F.Cu at (77.0, 82.4)
- C4: moved to B.Cu
- U1: footprint Wickerlib:TO-220-NEUTRAL123-VERT-LONGPADS -> Wickerlib:TO-220-NEUTRAL123-HORZ-LONGPADS
- moved C15 22.9 mm to (103.8, 83.1)
- moved R11 20.1 mm to (80.0, 78.8)
- moved C11 19.6 mm to (72.1, 82.5), turned to 270 degrees
- moved R13 19.0 mm to (80.1, 106.3), turned to 90 degrees
- moved J5 16.9 mm to (64.8, 80.6)
- moved C8 14.6 mm to (65.6, 59.1), turned to 180 degrees
- moved U2 14.2 mm to (68.0, 91.4), turned to 270 degrees
- moved Q1 13.9 mm to (83.2, 81.9), turned to 270 degrees
- moved C4 13.1 mm to (69.2, 69.2), turned to 180 degrees
- moved C12 13.0 mm to (82.5, 88.3), turned to 0 degrees
- moved D2 13.0 mm to (83.9, 92.2), turned to 270 degrees
- moved C16 12.7 mm to (66.7, 85.5), turned to 180 degrees
- moved D3 12.1 mm to (69.0, 114.2), turned to 0 degrees
- moved C5 9.32 mm to (93.3, 79.4), turned to 180 degrees
- moved R12 8.87 mm to (76.6, 97.2)
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Routing:
- net Net-(C15-Pad1): track 30.5 -> 10.3 mm
- net GND: track 0.00 -> 16.5 mm
- net Net-(C6-Pad1): track 70.5 -> 54.5 mm, vias 0 -> 3
- net Net-(C16-Pad1): track 26.8 -> 13.4 mm, vias 1 -> 0
- net Net-(D3-Pad2): track 14.3 -> 26.9 mm
- net Net-(BNC1-Pad1): track 34.2 -> 21.9 mm
- net Net-(BNC3-Pad1): track 11.5 -> 23.3 mm
- net Net-(C13-Pad1): track 22.0 -> 33.3 mm, vias 1 -> 2
- net Net-(C3-Pad1): track 73.7 -> 63.5 mm, vias 3 -> 0
- net Net-(D2-Pad1): track 7.13 -> 17.3 mm
- net +9V: track 47.9 -> 57.5 mm, vias 2 -> 0
- net +2V: track 29.5 -> 20.4 mm
- net Net-(C4-Pad2): track 15.2 -> 6.24 mm
- net Net-(C5-Pad2): track 41.8 -> 33.0 mm
- net (no net): track 7.62 -> 0.00 mm
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Other:
- board text added: "12/ 18V"
- board text added: "9V INPUT"
- board text added: "ANT_IN"
- board text added: "AUDIO"
- board text added: "FILTER"
- board text added: "LINE IN/OUT"
- board text added: "v1.3"
- board text added: "v1.3 12/26/2016"
- board text removed: "v1.2"
- board text removed: "v1.2 12/9/2016"
