File: e202var-vlf-radio-receiver.kicad_pcb (KiCad board)
At the start: 2 copper layers, 55.9 x 81.3 mm, 53 parts, among them J1 9V, J2 ON/OFF, J3 HEADPHONES, J4 12V/18V, J5 FILTER, Q1 BC547, Q2 BC547, U1 MC7809, U2 TLE2426, U3 NJM386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

Commit message: Fixed several schematic issues.
Parts:
- removed C8: 150pF, Wickerlib:CAP-DISC-D3MM-P2.5MM
- removed H1, H2, H3: HOLE-PLATED-3.2MM, Wickerlib:HOLE-PLATED-3.2MM
- removed R14: 2.2K, Wickerlib:RES-CARBONFILM-7MM
- removed SMA1: ANT IN, Wickerlib:CONN-SMA-STRAIGHT-TH
- added C14: 22nF, Wickerlib:CAP-DISC-D3MM-P2.5MM, F.Cu at (65.6, 59.1)
- C15: value 150pF -> 22nF
- moved C15 0.74 mm to (103.8, 83.9)
Connections:
- C3 pad 2: Net-(C3-Pad2) -> +2V
- R1 pad 2: Net-(C3-Pad2) -> +2V
- U3 pad 2: Net-(C6-Pad1) -> Net-(C15-Pad1)
- U3 pad 3: Net-(U3-Pad3) -> GND
- U3 pad 4: Net-(U3-Pad3) -> GND
Routing:
- net Net-(C15-Pad1): track 10.3 -> 51.8 mm
- net +2V: track 20.4 -> 55.7 mm
- net Net-(D3-Pad2): track 26.9 -> 10.1 mm
- net Net-(C3-Pad2): track 12.8 -> 0.00 mm
- net +9V: track 57.5 -> 67.7 mm, vias 0 -> 1
- net Net-(C6-Pad1): track 54.5 -> 44.8 mm
- net Net-(U3-Pad3): track 2.54 -> 0.00 mm
- net Net-(BNC2-Pad1): track 27.2 -> 25.7 mm
- net GND: track 16.5 -> 15.7 mm
Other:
- board text added: "E202VAR"
- board text added: "v1.4"
- board text added: "v1.4 2/23/2017"
- board text removed: "v1.3 12/26/2016"
