File: e202var-vlf-radio-receiver.kicad_pcb (KiCad board)
At the start: 2 copper layers, 55.9 x 81.3 mm, 48 parts, among them J1 9V, J2 ON/OFF, J3 HEADPHONES, J4 12V/18V, J5 FILTER, Q1 BC547, Q2 BC547, U1 MC7809, U2 TLE2426, U3 NJM386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

Commit message: Added three mounting holes to v1.4. Release.
Parts:
- added H1: HOLE-PLATED-3.2MM, Wickerlib:HOLE-PLATED-3.2MM, F.Cu at (95.2, 41.9)
- added H2: HOLE-PLATED-3.2MM, Wickerlib:HOLE-PLATED-3.2MM, F.Cu at (63.5, 41.9)
- added H3: HOLE-PLATED-3.2MM, Wickerlib:HOLE-PLATED-3.2MM, F.Cu at (63.5, 114.3)
Routing:
- net Net-(BNC2-Pad1): track 25.7 -> 24.7 mm
Changed lines of the file:
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@@
     (links 92)
     (no_connects 0)
-    (area 57.848759 33.5026 178.510001 123.746001)
+    (area 55.103143 33.5026 178.510001 123.746001)
     (thickness 1.6)
     (drawings 40)
-    (tracks 245)
+    (tracks 246)
     (zones 0)
-    (modules 48)
+    (modules 51)
     (nets 31)
   )
@@
     (title "E202VAR Natural Radio Receiver")
     (date "16 Oct 2015")
-    (rev "v1.4")
+    (rev v1.4)
     (company "CERN Open Hardware License v1.2")
-    (comment 1 "jenner@wickerbox.net")
-    (comment 2 "http://wickerbox.net")
+    (comment 1 jenner@wickerbox.net)
+    (comment 2 http://wickerbox.net)
     (comment 3 "Wickerbox Electronics")
   )
@@
       (net 17 "Net-(C10-Pad1)"))
   )
+  (module Wickerlib:HOLE-PLATED-3.2MM (layer F.Cu)
+    (at 63.5 41.91)
+    (fp_text reference H2 (at 0 0) (layer F.Fab)
+      (effects (font (size 1 1) (thickness 0.15)))
+    )
+    (fp_text value HOLE-PLATED-3.2MM (at 0 -0.5) (layer F.Fab) hide
+      (effects (font (size 1 1) (thickness 0.15)))
+    )
+    (fp_circle (center 0 0) (end 2.54 1.27) (layer F.Fab) (width 0.04064))
+    (pad 1 thru_hole circle (at 0 0) (size 5 5) (drill 3.2) (layers *.Cu *.Mask))
+  )
+  (module Wickerlib:HOLE-PLATED-3.2MM (layer F.Cu)
+    (at 63.5 114.3)
+    (fp_text reference H3 (at 0 0) (layer F.Fab)
+      (effects (font (size 1 1) (thickness 0.15)))
+    )
+    (fp_text value HOLE-PLATED-3.2MM (at 0 -0.5) (layer F.Fab) hide
+      (effects (font (size 1 1) (thickness 0.15)))
+    )
+    (fp_circle (center 0 0) (end 2.54 1.27) (layer F.Fab) (width 0.04064))
+    (pad 1 thru_hole circle (at 0 0) (size 5 5) (drill 3.2) (layers *.Cu *.Mask))
+  )
+  (module Wickerlib:HOLE-PLATED-3.2MM (layer F.Cu)
+    (at 95.25 41.91)
+    (fp_text reference H1 (at 0 0) (layer F.Fab)
+      (effects (font (size 1 1) (thickness 0.15)))
+    )
+    (fp_text value HOLE-PLATED-3.2MM (at 0 -0.5) (layer F.Fab) hide
+      (effects (font (size 1 1) (thickness 0.15)))
+    )
+    (fp_circle (center 0 0) (end 2.54 1.27) (layer F.Fab) (width 0.04064))
+    (pad 1 thru_hole circle (at 0 0) (size 5 5) (drill 3.2) (layers *.Cu *.Mask))
+  )
   (module Wickerlib:RES-CARBONFILM-7MM (layer F.Cu)
     (at 97.3455 70.485 270)
@@
       (net 1 GND))
   )
-  (gr_text v1.4 (at 94.6404 44.2595) (layer F.SilkS)
+  (gr_text v1.4 (at 89.1032 43.4721) (layer F.SilkS)
     (effects (font (thickness 0.254)))
   )
-  (gr_text E202VAR (at 89.7001 41.3258) (layer F.SilkS)
-    (effects (font (size 2.286 2.286) (thickness 0.508)))
+  (gr_text E202VAR (at 86.6267 40.8432) (layer F.SilkS)
+    (effects (font (thickness 0.254)))
   )
   (gr_text "9V INPUT" (at 62.6745 108.5215) (layer F.SilkS)
@@
   (segment (start 98.199842 110.998) (end 100.28174 110.998) (width 0.508) (layer F.Cu) (net 2))
   (segment (start 96.724102 109.52226) (end 98.199842 110.998) (width 0.508) (layer F.Cu) (net 2))
-  (segment (start 78.74 44.704) (end 94.996 44.704) (width 0.508) (layer F.Cu) (net 3))
+  (segment (start 93.7514 46.482) (end 80.518 46.482) (width 0.508) (layer F.Cu) (net 3))
+  (segment (start 80.518 46.482) (end 78.74 44.704) (width 0.508) (layer F.Cu) (net 3))
+  (segment (start 94.99092 47.72152) (end 93.7514 46.482) (width 0.508) (layer F.Cu) (net 3))
+  (segment (start 96.39808 47.72152) (end 94.99092 47.72152) (width 0.508) (layer F.Cu) (net 3))
   (segment (start 96.52 47.752) (end 99.69754 47.752) (width 0.508) (layer F.Cu) (net 3))
-  (segment (start 94.996 44.704) (end 96.52 46.228) (width 0.508) (layer F.Cu) (net 3))
-  (segment (start 96.52 46.228) (end 96.52 47.752) (width 0.508) (layer F.Cu) (net 3))
   (segment (start 99.69754 47.752) (end 101.20376 46.24578) (width 0.508) (layer F.Cu) (net 3))
   (segment (start 101.20376 46.24578) (end 101.65334 46.24578) (width 0.508) (layer F.Cu) (net 3))

Commit message: Release v1.4. Verified build. Project complete.
Parts:
- moved C1 11.6 mm to (72.9, 96.0)
- moved C10 11.6 mm to (108.3, 72.1)
- moved C12 11.6 mm to (92.8, 93.8)
- moved C15 11.6 mm to (114.0, 89.4)
- moved C3 11.6 mm to (71.7, 69.6)
- moved C4 11.6 mm to (79.4, 74.8)
- moved C6 11.6 mm to (113.4, 76.8)
- moved C7 11.6 mm to (112.4, 80.2)
- moved D2 11.6 mm to (94.1, 97.8)
- moved D3 11.6 mm to (79.2, 119.7)
- moved H1 11.6 mm to (105.5, 47.5)
- moved H2 11.6 mm to (73.7, 47.5)
- moved H3 11.6 mm to (73.7, 119.9)
- moved J2 11.6 mm to (89.3, 119.4)
- moved J4 11.6 mm to (101.6, 115.1)
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Connections:
- U1 pad 1: GND -> Net-(D2-Pad1)
- U1 pad 2: +9V -> GND
- U1 pad 3: Net-(D2-Pad1) -> +9V
Routing:
- net +9V: track 67.7 -> 55.7 mm, vias 1 -> 0
- net GND: track 15.7 -> 21.9 mm, vias 0 -> 1
- net Net-(D2-Pad1): track 17.3 -> 15.1 mm
Other:
- board text added: "FABRICATION NOTES 1. THIS IS A 2 LAYER BOARD. 2. EXTERNAL LAYERS SHALL HAVE 1 OZ COPPER. 3. MATERIAL: FR4 AND 0.062 INCH +/- 10% THICK. 4. BOARDS SHALL BE ROHS COMPLIANT. 5. MANUFACTURE IN ACCORDANCE WITH IPC-6012 CLASS 2 6. MASK: BOTH SIDES OF THE BOARD SHALL HAVE SOLDER MASK (ANY COLOR) OVER BARE COPPER. 7. SILK: BOTH SIDES OF THE BOARD SHALL HAVE WHITE SILK. DO NOT PLACE SILK OVER BARE COPPER.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"
- board text removed: "E202VAR VLF Natural Radio Receiver"
- board text removed: "v1.3"
- board text removed: "v1.4 2/23/2017"
