File: e202var-vlf-radio-receiver.sch (KiCad schematic (older format))
At the start: 48 parts, among them J1 9V, J2 ON/OFF, J3 HEADPHONES, J4 12V/18V, J5 FILTER, Q1 BC547, Q2 BC547, U1 MC7809, U2 TLE2426, U3 NJM386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

Commit message: Release v1.4. Verified build. Project complete.
Parts:
- C14, C15: S1_PN 399-14089-2-ND -> 399-14089-1-ND
Changed lines of the file:
@@
 F 6 "C315C223K5R5TA7303" H 8075 3575 50  0001 C CIN "MF_PN"
 F 7 "Digikey" H 8075 3575 50  0001 C CIN "S1_Name"
-F 8 "399-14089-2-ND" H 8075 3575 50  0001 C CIN "S1_PN"
+F 8 "399-14089-1-ND" H 8075 3575 50  0001 C CIN "S1_PN"
 	1    8075 3925
 	1    0    0    -1
@@
 F 6 "C315C223K5R5TA7303" H 8600 3575 50  0001 C CIN "MF_PN"
 F 7 "Digikey" H 8600 3575 50  0001 C CIN "S1_Name"
-F 8 "399-14089-2-ND" H 8600 3575 50  0001 C CIN "S1_PN"
+F 8 "399-14089-1-ND" H 8600 3575 50  0001 C CIN "S1_PN"
 	1    8600 3925
 	1    0    0    -1
